Commit message: Added non collisions for the new probing tool

File: config/hand.xacro (robot description, xacro)
@@ -11,6 +11,10 @@
       <link name="panda_leftfinger" />
       <link name="panda_rightfinger" />
+      <link name="panda_probe_cyl" />
+      <link name="panda_probe_ball" />
       <joint name="panda_finger_joint1" />
-      <passive_joint name="panda_finger_joint2" />
+      <joint name="panda_finger_joint2" />
+      <joint name="panda_probe_ball_joint" />
+      <joint name="panda_probe_cyl_joint" />
     </group>
     <!--GROUP STATES: Purpose: Define a named state for a particular group, in terms of joint values. This is useful to define states like 'folded arms'-->
@@ -19,5 +23,9 @@
     <disable_collisions link1="panda_hand" link2="panda_leftfinger" reason="Adjacent" />
     <disable_collisions link1="panda_hand" link2="panda_rightfinger" reason="Adjacent" />
+    <disable_collisions link1="panda_hand" link2="panda_probe_cyl" reason="Adjacent" />
+    <disable_collisions link1="panda_probe_cyl" link2="panda_probe_ball" reason="Adjacent" />
     <disable_collisions link1="panda_leftfinger" link2="panda_rightfinger" reason="Default" />
+    <disable_collisions link1="panda_leftfinger" link2="panda_probe_cyl" reason="Default" />
+    <disable_collisions link1="panda_rightfinger" link2="panda_probe_cyl" reason="Default" />
   </xacro:macro>
 </robot>
